Commit message: ADD: GAZEBO model define and control code

File: src/robot_description/urdf/dual_motion_robot_drive/dual_motion_robot.xacro (robot description, xacro)
@@ -1,12 +1,12 @@
 <?xml version="1.0" ?>
 <robot name="dual_motion_robot" xmlns:xacro="http://www.ros.org/wiki/xacro">
-  <xacro:include filename="$(find robot_description)/urdf/dual_motion_robot/materials.xacro" />
-  <xacro:include filename="$(find robot_description)/urdf/dual_motion_robot/dual_motion_robot.gazebo" />
-  <xacro:include filename="$(find robot_description)/urdf/dual_motion_robot/macros.xacro" />
-  <xacro:include filename="$(find robot_description)/urdf/dual_motion_robot/dual_motion_robot_transmision.xacro" />
+  <xacro:include filename="$(find robot_description)/urdf/dual_motion_robot_drive/materials.xacro" />
+  <xacro:include filename="$(find robot_description)/urdf/dual_motion_robot_drive/dual_motion_robot.gazebo" />
+  <xacro:include filename="$(find robot_description)/urdf/dual_motion_robot_drive/macros.xacro" />
+  <xacro:include filename="$(find robot_description)/urdf/dual_motion_robot_drive/dual_motion_robot_transmision.xacro" />
   <link name="link_chassis">
     <!-- pose and inertial -->
     <inertial>
-      <mass value="20"/>
+      <mass value="10"/>
       <origin rpy="0 0 0" xyz="0 0 0"/>
       <inertia ixx="0.0395416666667" ixy="0" ixz="0" iyy="0.106208333333" iyz="0" izz="0.106208333333"/>
@@ -30,5 +30,5 @@
     <pose>0 0 0.1 0 0 0</pose>
     <inertial>
-      <mass value="0.001"/>
+      <mass value="5"/>
       <origin rpy="0 0 0" xyz="0 0 0.1"/>
       <inertia ixx="0.0395416666667" ixy="0" ixz="0" iyy="0.106208333333" iyz="0" izz="0.106208333333"/>
@@ -50,8 +50,6 @@
   <xacro:link_wheel name="link_right_wheel" />
   <xacro:joint_wheel name="wheel_R_joint" child="link_right_wheel" origin_xyz="0 0.20 -0.1" />
-  <xacro:SimpleTransmissionVeolcity n="1" joint="wheel_R_joint" />
   <xacro:link_wheel name="link_left_wheel" />
   <xacro:joint_wheel name="wheel_L_joint" child="link_left_wheel" origin_xyz="0 -0.20 -0.1" />
-  <xacro:SimpleTransmissionVeolcity n="1" joint="wheel_L_joint" />
   <xacro:base_joint name="chassis_pos_joint" child="link_chassis" origin_xyz="0 0 0.11" />
 </robot>

File: src/robot_description/urdf/dual_motion_robot_drive/macros.xacro (robot description, xacro)
@@ -4,5 +4,5 @@
         <link name="${name}">
             <inertial>
-              <mass value="5"/>
+              <mass value="3"/>
               <origin rpy="0 1.5707 1.5707" xyz="0 0 0"/>
               <inertia ixx="0.000526666666667" ixy="0" ixz="0" iyy="0.000526666666667" iyz="0" izz="0.001"/>

Commit message: EDIT: mpc code continuous -> discrete

File: src/robot_description/urdf/dual_motion_robot_drive/dual_motion_robot.xacro (robot description, xacro)
@@ -10,10 +10,10 @@
       <mass value="10"/>
       <origin rpy="0 0 0" xyz="0 0 0"/>
-      <inertia ixx="0.0395416666667" ixy="0" ixz="0" iyy="0.106208333333" iyz="0" izz="0.106208333333"/>
+      <inertia ixx="0.2124" ixy="0" ixz="0" iyy="0.2124" iyz="0" izz="0.4166"/>
     </inertial>
     <!-- body -->
     <collision name="collision_chassis">
       <geometry>
-        <box size="0.7 0.7 0.07"/>
+        <box size="0.5 0.5 0.07"/>
       </geometry>
     </collision>
@@ -21,5 +21,5 @@
       <origin rpy="0 0 0" xyz="0 0 0"/>
       <geometry>
-        <box size="0.7 0.7 0.07"/>
+        <box size="0.5 0.5 0.07"/>
       </geometry>
       <material name="blue"/>
@@ -37,5 +37,5 @@
     <collision name="collision_wheel_link">
       <geometry>
-        <box size="0.07 0.4 0.2"/>
+        <box size="0.07 0.4 0.5"/>
       </geometry>
     </collision>
@@ -43,5 +43,5 @@
       <origin rpy="0 0 0" xyz="0 0 0"/>
       <geometry>
-        <box size="0.07 0.4 0.2"/>
+        <box size="0.07 0.4 0.5"/>
       </geometry>
       <material name="blue"/>
@@ -49,7 +49,7 @@
   </link>
   <xacro:link_wheel name="link_right_wheel" />
-  <xacro:joint_wheel name="wheel_R_joint" child="link_right_wheel" origin_xyz="0 0.20 -0.1" />
+  <xacro:joint_wheel name="wheel_R_joint" child="link_right_wheel" origin_xyz="0 0.20 -0.25" />
   <xacro:link_wheel name="link_left_wheel" />
-  <xacro:joint_wheel name="wheel_L_joint" child="link_left_wheel" origin_xyz="0 -0.20 -0.1" />
-  <xacro:base_joint name="chassis_pos_joint" child="link_chassis" origin_xyz="0 0 0.11" />
+  <xacro:joint_wheel name="wheel_L_joint" child="link_left_wheel" origin_xyz="0 -0.20 -0.25" />
+  <xacro:base_joint name="chassis_pos_joint" child="link_chassis" origin_xyz="0 0 0.26" />
 </robot>

Commit message: EDIT: mpc code

File: src/robot_description/urdf/dual_motion_robot_drive/dual_motion_robot.xacro (robot description, xacro)
@@ -15,5 +15,5 @@
     <collision name="collision_chassis">
       <geometry>
-        <box size="0.5 0.5 0.07"/>
+        <box size="0.5 0.5 0.05"/>
       </geometry>
     </collision>
@@ -21,5 +21,5 @@
       <origin rpy="0 0 0" xyz="0 0 0"/>
       <geometry>
-        <box size="0.5 0.5 0.07"/>
+        <box size="0.5 0.5 0.05"/>
       </geometry>
       <material name="blue"/>
@@ -37,5 +37,5 @@
     <collision name="collision_wheel_link">
       <geometry>
-        <box size="0.07 0.4 0.5"/>
+        <box size="0.07 0.4 0.2"/>
       </geometry>
     </collision>
@@ -43,5 +43,5 @@
       <origin rpy="0 0 0" xyz="0 0 0"/>
       <geometry>
-        <box size="0.07 0.4 0.5"/>
+        <box size="0.07 0.4 0.2"/>
       </geometry>
       <material name="blue"/>
@@ -49,7 +49,7 @@
   </link>
   <xacro:link_wheel name="link_right_wheel" />
-  <xacro:joint_wheel name="wheel_R_joint" child="link_right_wheel" origin_xyz="0 0.20 -0.25" />
+  <xacro:joint_wheel name="wheel_R_joint" child="link_right_wheel" origin_xyz="0 0.20 -0.1" />
   <xacro:link_wheel name="link_left_wheel" />
-  <xacro:joint_wheel name="wheel_L_joint" child="link_left_wheel" origin_xyz="0 -0.20 -0.25" />
-  <xacro:base_joint name="chassis_pos_joint" child="link_chassis" origin_xyz="0 0 0.26" />
+  <xacro:joint_wheel name="wheel_L_joint" child="link_left_wheel" origin_xyz="0 -0.20 -0.1" />
+  <xacro:base_joint name="chassis_pos_joint" child="link_chassis" origin_xyz="0 0 0.1" />
 </robot>

File: src/robot_description/urdf/dual_motion_robot_drive/macros.xacro (robot description, xacro)
@@ -6,5 +6,5 @@
               <mass value="3"/>
               <origin rpy="0 1.5707 1.5707" xyz="0 0 0"/>
-              <inertia ixx="0.000526666666667" ixy="0" ixz="0" iyy="0.000526666666667" iyz="0" izz="0.001"/>
+              <inertia ixx="0.0115" ixy="0" ixz="0" iyy="0.0115" iyz="0" izz="0.15"/>
             </inertial>
             <collision name="link_right_wheel_collision">
@@ -43,5 +43,5 @@
         <parent link="wheel_link"/>
         <axis rpy="0 0 0" xyz="1 0 0"/>
-        <limit effort="10" lower="-0.35" upper="0.35" velocity="0.1" />
+        <!-- <limit effort="10" lower="-0.35" upper="0.35" velocity="0.1" /> -->
       </joint>
     </xacro:macro>

Commit message: EDIT: MPC code

File: src/robot_description/urdf/dual_motion_robot_drive/dual_motion_robot.xacro (robot description, xacro)
@@ -37,4 +37,5 @@
     <collision name="collision_wheel_link">
       <geometry>
+        <!-- <box size="0.07 0.4 0.4"/> -->
         <box size="0.07 0.4 0.2"/>
       </geometry>
@@ -44,4 +45,5 @@
       <geometry>
         <box size="0.07 0.4 0.2"/>
+        <!-- <box size="0.07 0.4 0.4"/> -->
       </geometry>
       <material name="blue"/>
@@ -50,6 +52,9 @@
   <xacro:link_wheel name="link_right_wheel" />
   <xacro:joint_wheel name="wheel_R_joint" child="link_right_wheel" origin_xyz="0 0.20 -0.1" />
+  <!-- <xacro:joint_wheel name="wheel_R_joint" child="link_right_wheel" origin_xyz="0 0.20 -0.2" /> -->
   <xacro:link_wheel name="link_left_wheel" />
+  <!-- <xacro:joint_wheel name="wheel_L_joint" child="link_left_wheel" origin_xyz="0 -0.20 -0.2" /> -->
   <xacro:joint_wheel name="wheel_L_joint" child="link_left_wheel" origin_xyz="0 -0.20 -0.1" />
   <xacro:base_joint name="chassis_pos_joint" child="link_chassis" origin_xyz="0 0 0.1" />
+  <!-- <xacro:base_joint name="chassis_pos_joint" child="link_chassis" origin_xyz="0 0 0.2" /> -->
 </robot>
