Commit message: EDIT: MPC Continuous model code

File: src/robot_description/urdf/dual_motion_robot_drive/macros.xacro (robot description, xacro)
@@ -4,5 +4,5 @@
         <link name="${name}">
             <inertial>
-              <mass value="3"/>
+              <mass value="1"/>
               <origin rpy="0 1.5707 1.5707" xyz="0 0 0"/>
               <inertia ixx="0.0115" ixy="0" ixz="0" iyy="0.0115" iyz="0" izz="0.15"/>
